File: PF_Contro_PCB/PF_Contro_PCB.kicad_pcb (KiCad board)
At the start: 4 copper layers, 100 x 60 mm, 140 parts, among them Q1 DMP4015SPSQ-13, U1 UCC27524ADR, U2 ADS1115IDGSR, U3 ADS1115IDGSR, U4 TPS62162DSG, U5 UCC27524ADR, U6 TPS62163DSGR, U7 ESP32-S3-WROOM-1U-N16

Commit message: Test Commit
Parts:
- moved ACT4 7.02 mm to (74.0, 114.4)
Changed lines of the file:
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@@
 	(footprint "TerminalBlock_Phoenix:TerminalBlock_Phoenix_MKDS-1,5-2-5.08_1x02_P5.08mm_Horizontal"
 		(layer "F.Cu")
-		(at 78.3475 108.855)
+		(at 74.01 114.37)
 		(descr "Terminal Block Phoenix MKDS-1,5-2-5.08, 2 pins, pitch 5.08mm, size 10.2x9.8mm, drill diameter 1.3mm, pad diameter 2.6mm, http://www.farnell.com/datasheets/100425.pdf, script-generated using https://gitlab.com/kicad/libraries/kicad-footprint-generator/-/tree/master/scripts/TerminalBlock_Phoenix")
 		(tags "THT Terminal Block Phoenix MKDS-1,5-2-5.08 pitch 5.08mm size 10.2x9.8mm drill 1.3mm pad 2.6mm")

Commit message: Test
Parts:
- moved ACT4 8.17 mm to (82.0, 115.9)
Changed lines of the file:
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@@
 	(footprint "TerminalBlock_Phoenix:TerminalBlock_Phoenix_MKDS-1,5-2-5.08_1x02_P5.08mm_Horizontal"
 		(layer "F.Cu")
-		(at 74.01 114.37)
+		(at 82.045 115.8725)
 		(descr "Terminal Block Phoenix MKDS-1,5-2-5.08, 2 pins, pitch 5.08mm, size 10.2x9.8mm, drill diameter 1.3mm, pad diameter 2.6mm, http://www.farnell.com/datasheets/100425.pdf, script-generated using https://gitlab.com/kicad/libraries/kicad-footprint-generator/-/tree/master/scripts/TerminalBlock_Phoenix")
 		(tags "THT Terminal Block Phoenix MKDS-1,5-2-5.08 pitch 5.08mm size 10.2x9.8mm drill 1.3mm pad 2.6mm")
